File: Transformerless Inverter kicad schematics and PCB design/Transformerless inverter.kicad_pcb (KiCad board)
At the start: 2 copper layers, 40 parts

Commit message: made some changes to the inverter pcb and added battery combiner board
Parts:
- removed the REF** at (186.7, 171.4)
- removed the REF** at (232.4, 252.7)
- removed the REF** at (222.2, 280.7)
- removed the REF** at (232.4, 260.4)
- removed the REF** at (232.4, 275.6)
- removed the REF** at (204.5, 266.7)
- removed the REF** at (214.6, 256.5)
- removed the REF** at (233.7, 290.8)
- added REF**: TerminalBlock_4Ucon_1x08_P3.50mm_Horizontal, TerminalBlock_4Ucon:TerminalBlock_4Ucon_1x08_P3.50mm_Horizontal, F.Cu at (174.0, 167.6)
Routing:
- net (no net): track 4927.1 -> 4515.1 mm, vias 48 -> 46
